File: NixieKit - コピー.kicad_pcb (KiCad board)
At the start: 2 copper layers, 49 x 99.5 mm, 30 parts, among them J1 Conn_01x04, J10 Conn_01x12, J2 Conn_01x05, J3 Conn_01x04, J4 Conn_02x03_Odd_Even, J5 Conn_01x04, J6 Conn_01x05, J7 Conn_01x05, J8 CONN_01X05, J9 Conn_01x12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

Commit message: first gerber out
Routing:
- removed copper zone on B.Cu, net GND
- removed copper zone on F.Cu, net GND
